Commit message: style: improve Gazebo robot visual model

File: src/simulation_pkg/urdf/lekiwi_base.xacro (robot description, xacro)
@@ -5,15 +5,34 @@
     <!-- Base link -->
     <link name="${prefix}base_link">
-      <visual>
+      <visual name="base_body">
+        <origin xyz="0 0 0" rpy="0 0 0"/>
         <geometry>
-          <cylinder radius="0.2" length="0.1"/>
+          <box size="0.46 0.34 0.08"/>
         </geometry>
         <material name="dark_grey">
-          <color rgba="0.3 0.3 0.3 1.0"/>
+          <color rgba="0.25 0.25 0.25 1.0"/>
+        </material>
+      </visual>
+      <visual name="base_top_plate">
+        <origin xyz="0 0 0.055" rpy="0 0 0"/>
+        <geometry>
+          <cylinder radius="0.18" length="0.02"/>
+        </geometry>
+        <material name="medium_grey">
+          <color rgba="0.45 0.45 0.45 1.0"/>
+        </material>
+      </visual>
+      <visual name="front_marker">
+        <origin xyz="0.20 0 0.075" rpy="0 0 0"/>
+        <geometry>
+          <box size="0.08 0.04 0.03"/>
+        </geometry>
+        <material name="front_green">
+          <color rgba="0.0 0.8 0.25 1.0"/>
         </material>
       </visual>
       <collision>
         <geometry>
-          <cylinder radius="0.2" length="0.1"/>
+          <box size="0.46 0.34 0.08"/>
         </geometry>
       </collision>
@@ -26,7 +45,8 @@
     <xacro:macro name="omni_wheel" params="name angle">
       <link name="${prefix}${name}_wheel">
-        <visual>
+        <visual name="${name}_tire">
+          <origin xyz="0 0 0" rpy="${pi/2} 0 0"/>
           <geometry>
-            <cylinder radius="0.05" length="0.02"/>
+            <cylinder radius="0.065" length="0.04"/>
           </geometry>
           <material name="black">
@@ -34,7 +54,17 @@
           </material>
         </visual>
+        <visual name="${name}_hub">
+          <origin xyz="0 0 0" rpy="${pi/2} 0 0"/>
+          <geometry>
+            <cylinder radius="0.025" length="0.048"/>
+          </geometry>
+          <material name="wheel_hub">
+            <color rgba="0.8 0.8 0.8 1.0"/>
+          </material>
+        </visual>
         <collision>
+          <origin xyz="0 0 0" rpy="${pi/2} 0 0"/>
           <geometry>
-            <cylinder radius="0.05" length="0.02"/>
+            <cylinder radius="0.065" length="0.04"/>
           </geometry>
         </collision>
@@ -47,5 +77,5 @@
         <parent link="${prefix}base_link"/>
         <child link="${prefix}${name}_wheel"/>
-        <origin xyz="${0.15 * cos(angle)} ${0.15 * sin(angle)} -0.04" rpy="0 0 0"/>
+        <origin xyz="${0.23 * cos(angle)} ${0.23 * sin(angle)} -0.045" rpy="0 0 ${angle}"/>
         <axis xyz="0 1 0"/>
       </joint>
@@ -56,4 +86,13 @@
     <!-- IMU link -->
     <link name="${prefix}imu_link">
+      <visual name="imu_marker">
+        <origin xyz="0 0 0" rpy="0 0 0"/>
+        <geometry>
+          <box size="0.035 0.025 0.012"/>
+        </geometry>
+        <material name="imu_red">
+          <color rgba="0.9 0.05 0.05 1.0"/>
+        </material>
+      </visual>
       <inertial>
         <mass value="0.01"/>

File: src/simulation_pkg/urdf/lekiwi_full.urdf.xacro (robot description, xacro)
@@ -18,4 +18,9 @@
         <remapping>joint_states:=/joint_states</remapping>
       </ros>
+      <joint_name>front_wheel_joint</joint_name>
+      <joint_name>left_wheel_joint</joint_name>
+      <joint_name>right_wheel_joint</joint_name>
+      <joint_name>gimbal_yaw_joint</joint_name>
+      <joint_name>gimbal_pitch_joint</joint_name>
       <update_rate>100</update_rate>
     </plugin>

File: src/simulation_pkg/urdf/lekiwi_gimbal.xacro (robot description, xacro)
@@ -5,10 +5,20 @@
     <!-- Pan (yaw) link -->
     <link name="${prefix}gimbal_yaw_link">
-      <visual>
+      <visual name="yaw_base">
+        <origin xyz="0 0 0" rpy="0 0 0"/>
         <geometry>
-          <cylinder radius="0.06" length="0.05"/>
+          <cylinder radius="0.085" length="0.07"/>
         </geometry>
-        <material name="silver">
-          <color rgba="0.7 0.7 0.7 1.0"/>
+        <material name="gimbal_yaw_orange">
+          <color rgba="0.95 0.55 0.1 1.0"/>
+        </material>
+      </visual>
+      <visual name="yaw_upright">
+        <origin xyz="0 0 0.075" rpy="0 0 0"/>
+        <geometry>
+          <box size="0.035 0.13 0.12"/>
+        </geometry>
+        <material name="gimbal_side_orange">
+          <color rgba="0.95 0.55 0.1 1.0"/>
         </material>
       </visual>
@@ -21,5 +31,5 @@
       <parent link="${parent}"/>
       <child link="${prefix}gimbal_yaw_link"/>
-      <origin xyz="0 0 0.12" rpy="0 0 0"/>
+      <origin xyz="0 0 0.13" rpy="0 0 0"/>
       <axis xyz="0 0 1"/>
       <limit effort="10" velocity="6.28" lower="-3.14" upper="3.14"/>
@@ -27,9 +37,12 @@
     <!-- Tilt (pitch) link -->
     <link name="${prefix}gimbal_pitch_link">
-      <visual>
+      <visual name="pitch_bar">
+        <origin xyz="0.035 0 0" rpy="0 0 0"/>
         <geometry>
-          <box size="0.08 0.04 0.03"/>
+          <box size="0.16 0.055 0.05"/>
         </geometry>
-        <material name="silver"/>
+        <material name="gimbal_pitch_blue">
+          <color rgba="0.1 0.35 0.95 1.0"/>
+        </material>
       </visual>
       <inertial>
@@ -41,5 +54,5 @@
       <parent link="${prefix}gimbal_yaw_link"/>
       <child link="${prefix}gimbal_pitch_link"/>
-      <origin xyz="0 0 0.03" rpy="0 0 0"/>
+      <origin xyz="0 0 0.10" rpy="0 0 0"/>
       <axis xyz="0 1 0"/>
       <limit effort="5" velocity="3.14" lower="-1.57" upper="1.57"/>
@@ -47,10 +60,20 @@
     <!-- Camera link (mounted on pitch axis) -->
     <link name="${prefix}camera_link">
-      <visual>
+      <visual name="camera_body">
+        <origin xyz="0.045 0 0" rpy="0 0 0"/>
         <geometry>
-          <box size="0.04 0.02 0.02"/>
+          <box size="0.11 0.055 0.045"/>
         </geometry>
-        <material name="blue">
-          <color rgba="0.1 0.1 0.8 1.0"/>
+        <material name="camera_blue">
+          <color rgba="0.05 0.12 0.75 1.0"/>
+        </material>
+      </visual>
+      <visual name="camera_lens">
+        <origin xyz="0.11 0 0" rpy="0 ${pi/2} 0"/>
+        <geometry>
+          <cylinder radius="0.018" length="0.018"/>
+        </geometry>
+        <material name="lens_black">
+          <color rgba="0.02 0.02 0.02 1.0"/>
         </material>
       </visual>
@@ -63,5 +86,5 @@
       <parent link="${prefix}gimbal_pitch_link"/>
       <child link="${prefix}camera_link"/>
-      <origin xyz="0.03 0 0" rpy="0 0 0"/>
+      <origin xyz="0.11 0 0" rpy="0 0 0"/>
     </joint>
     <!-- Camera optical frame (ROS convention: z-forward, x-right, y-down) -->

Commit message: fix: align Gazebo target and visual materials

File: src/simulation_pkg/urdf/lekiwi_base.xacro (robot description, xacro)
@@ -23,13 +23,4 @@
         </material>
       </visual>
-      <visual name="front_marker">
-        <origin xyz="0.20 0 0.075" rpy="0 0 0"/>
-        <geometry>
-          <box size="0.08 0.04 0.03"/>
-        </geometry>
-        <material name="front_green">
-          <color rgba="0.0 0.8 0.25 1.0"/>
-        </material>
-      </visual>
       <collision>
         <geometry>
@@ -42,4 +33,31 @@
       </inertial>
     </link>
+    <!-- Separate link so Gazebo can keep the front marker green. -->
+    <link name="${prefix}front_marker_link">
+      <visual name="front_marker">
+        <origin xyz="0 0 0" rpy="0 0 0"/>
+        <geometry>
+          <box size="0.08 0.04 0.03"/>
+        </geometry>
+        <material name="front_green">
+          <color rgba="0.0 0.8 0.25 1.0"/>
+        </material>
+      </visual>
+      <inertial>
+        <mass value="0.01"/>
+        <inertia ixx="1e-6" iyy="1e-6" izz="1e-6" ixy="0" ixz="0" iyz="0"/>
+      </inertial>
+    </link>
+    <joint name="${prefix}front_marker_joint" type="fixed">
+      <parent link="${prefix}base_link"/>
+      <child link="${prefix}front_marker_link"/>
+      <origin xyz="0.20 0 0.075" rpy="0 0 0"/>
+    </joint>
+    <gazebo reference="${prefix}base_link">
+      <material>Gazebo/DarkGrey</material>
+    </gazebo>
+    <gazebo reference="${prefix}front_marker_link">
+      <material>Gazebo/Green</material>
+    </gazebo>
     <!-- Omni wheels (3x, at 120° intervals) -->
     <xacro:macro name="omni_wheel" params="name angle">
@@ -80,4 +98,7 @@
         <axis xyz="0 1 0"/>
       </joint>
+      <gazebo reference="${prefix}${name}_wheel">
+        <material>Gazebo/Black</material>
+      </gazebo>
     </xacro:macro>
     <xacro:omni_wheel name="front" angle="${0}"/>
@@ -105,4 +126,7 @@
       <origin xyz="0 0 0.05" rpy="0 0 0"/>
     </joint>
+    <gazebo reference="${prefix}imu_link">
+      <material>Gazebo/Red</material>
+    </gazebo>
   </xacro:macro>
 </robot>

File: src/simulation_pkg/urdf/lekiwi_gimbal.xacro (robot description, xacro)
@@ -28,4 +28,7 @@
       </inertial>
     </link>
+    <gazebo reference="${prefix}gimbal_yaw_link">
+      <material>Gazebo/Orange</material>
+    </gazebo>
     <joint name="${prefix}gimbal_yaw_joint" type="revolute">
       <parent link="${parent}"/>
@@ -51,4 +54,7 @@
       </inertial>
     </link>
+    <gazebo reference="${prefix}gimbal_pitch_link">
+      <material>Gazebo/Blue</material>
+    </gazebo>
     <joint name="${prefix}gimbal_pitch_joint" type="revolute">
       <parent link="${prefix}gimbal_yaw_link"/>
@@ -83,4 +89,7 @@
       </inertial>
     </link>
+    <gazebo reference="${prefix}camera_link">
+      <material>Gazebo/Blue</material>
+    </gazebo>
     <joint name="${prefix}camera_joint" type="fixed">
       <parent link="${prefix}gimbal_pitch_link"/>
