Commit message: feat: 完善云台-底盘协同控制及仿真目标变换
- target_simulator: 修复 transform_to_camera_frame() 完整运动学链
  (odom→base_link→yaw→pitch→camera→optical), 使用 EntityState API
- platform_manager: 订阅 joint_states 提取云台角度, 发布到 PlatformState
- control_allocator: 新增云台限位感知的动态分配 (yaw/pitch saturation)
- pbvs_controller: 使用 Target.position 重建3D位姿, 加入方向估计
- gazebo.launch.py: 补全 gzserver 系统插件 (init/state/factory)
- lekiwi_gimbal.xacro: 视觉颜色调整 (orange→cyan, blue→magenta)

File: src/simulation_pkg/urdf/lekiwi_gimbal.xacro (robot description, xacro)
@@ -10,6 +10,6 @@
           <cylinder radius="0.085" length="0.07"/>
         </geometry>
-        <material name="gimbal_yaw_orange">
-          <color rgba="0.95 0.55 0.1 1.0"/>
+        <material name="gimbal_yaw_cyan">
+          <color rgba="0.0 0.9 0.9 1.0"/>
         </material>
       </visual>
@@ -19,6 +19,6 @@
           <box size="0.035 0.13 0.12"/>
         </geometry>
-        <material name="gimbal_side_orange">
-          <color rgba="0.95 0.55 0.1 1.0"/>
+        <material name="gimbal_side_cyan">
+          <color rgba="0.0 0.9 0.9 1.0"/>
         </material>
       </visual>
@@ -29,5 +29,5 @@
     </link>
     <gazebo reference="${prefix}gimbal_yaw_link">
-      <material>Gazebo/Orange</material>
+      <material>Gazebo/Cyan</material>
     </gazebo>
     <joint name="${prefix}gimbal_yaw_joint" type="revolute">
@@ -45,6 +45,6 @@
           <box size="0.16 0.055 0.05"/>
         </geometry>
-        <material name="gimbal_pitch_blue">
-          <color rgba="0.1 0.35 0.95 1.0"/>
+        <material name="gimbal_pitch_magenta">
+          <color rgba="0.95 0.1 0.7 1.0"/>
         </material>
       </visual>
@@ -55,5 +55,5 @@
     </link>
     <gazebo reference="${prefix}gimbal_pitch_link">
-      <material>Gazebo/Blue</material>
+      <material>Gazebo/Magenta</material>
     </gazebo>
     <joint name="${prefix}gimbal_pitch_joint" type="revolute">
