Commit message: v2.2

File: src/simulation_pkg/urdf/lekiwi_full.urdf.xacro (robot description, xacro)
@@ -2,4 +2,5 @@
 <!-- LEKIWI Full Robot: base + gimbal + sensors -->
 <robot name="lekiwi_fcr" xmlns:xacro="http://www.ros.org/wiki/xacro">
+  <xacro:arg name="enable_depth_camera" default="false"/>
   <!-- Include sub-models -->
   <xacro:include filename="lekiwi_base.xacro"/>
@@ -11,5 +12,5 @@
   <xacro:lekiwi_gimbal parent="base_link" prefix=""/>
   <!-- Instantiate sensors -->
-  <xacro:lekiwi_sensors parent="base_link" prefix=""/>
+  <xacro:lekiwi_sensors parent="base_link" prefix="" enable_depth_camera="$(arg enable_depth_camera)"/>
   <!-- Gazebo plugin: joint state publisher (TF + RViz updates for all joints) -->
   <gazebo>

File: src/simulation_pkg/urdf/lekiwi_sensors.xacro (robot description, xacro)
@@ -2,34 +2,36 @@
 <!-- LEKIWI Sensors: depth camera, LiDAR, IMU -->
 <robot xmlns:xacro="http://www.ros.org/wiki/xacro">
-  <xacro:macro name="lekiwi_sensors" params="parent:=base_link prefix:=''">
+  <xacro:macro name="lekiwi_sensors" params="parent:=base_link prefix:='' enable_depth_camera:=false">
     <!-- Depth camera (RGBD) — attached to camera_link via gimbal -->
-    <gazebo reference="${prefix}camera_optical_link">
-      <sensor type="depth" name="depth_camera">
-        <update_rate>30.0</update_rate>
-        <camera>
-          <horizontal_fov>1.20428</horizontal_fov>  <!-- 69° HFOV for OAK-D -->
-          <image>
-            <width>640</width>
-            <height>480</height>
-            <format>R8G8B8</format>
-          </image>
-          <clip>
-            <near>0.1</near>
-            <far>100.0</far>
-          </clip>
-        </camera>
-        <plugin name="camera_plugin" filename="libgazebo_ros_camera.so">
-          <ros>
-            <namespace>/camera</namespace>
-            <remapping>image_raw:=image_raw</remapping>
-            <remapping>camera_info:=camera_info</remapping>
-            <remapping>depth/image_raw:=depth/image_raw</remapping>
-          </ros>
-          <camera_name>camera</camera_name>
-          <frame_name>camera_optical_link</frame_name>
-          <hack_baseline>0.075</hack_baseline>
-        </plugin>
-      </sensor>
-    </gazebo>
+    <xacro:if value="${enable_depth_camera}">
+      <gazebo reference="${prefix}camera_optical_link">
+        <sensor type="depth" name="depth_camera">
+          <update_rate>30.0</update_rate>
+          <camera>
+            <horizontal_fov>1.20428</horizontal_fov>  <!-- 69° HFOV for OAK-D -->
+            <image>
+              <width>640</width>
+              <height>480</height>
+              <format>R8G8B8</format>
+            </image>
+            <clip>
+              <near>0.1</near>
+              <far>100.0</far>
+            </clip>
+          </camera>
+          <plugin name="camera_plugin" filename="libgazebo_ros_camera.so">
+            <ros>
+              <namespace>/camera</namespace>
+              <remapping>image_raw:=image_raw</remapping>
+              <remapping>camera_info:=camera_info</remapping>
+              <remapping>depth/image_raw:=depth/image_raw</remapping>
+            </ros>
+            <camera_name>camera</camera_name>
+            <frame_name>camera_optical_link</frame_name>
+            <hack_baseline>0.075</hack_baseline>
+          </plugin>
+        </sensor>
+      </gazebo>
+    </xacro:if>
     <!-- IMU sensor -->
     <gazebo reference="${prefix}imu_link">
